File: 02-wsg/esp32s3/esp32s3.kicad_sch (KiCad schematic)
At the start: 7 parts, among them U1 ESP32-S3, Y1 ECS-400-10-37B2-CKY-TR

Commit message: esp32s3 integration done
Parts:
- added AE1: Antenna_Chip, wsg_fp:XDCR_2450AT18B100E, symbol Device:Antenna_Chip
- added C10, C11, C14, C15, C7, C9: 0.1uF, Capacitor_SMD:C_0402_1005Metric, symbol Device:C
- added C12, C13: 17pF, Capacitor_SMD:C_0402_1005Metric, symbol Device:C
- added C5: 1.2pF, Capacitor_SMD:C_0201_0603Metric, symbol Device:C
- added C6: 4.7uF, Capacitor_SMD:C_0402_1005Metric, symbol Device:C
- added C8: 10uF, Capacitor_SMD:C_0402_1005Metric, symbol Device:C
- added IC2: W25N04KVZEIR, wsg_fp:SON127P800X600X80-9N-D, symbol wsg_syms:W25N04KVZEIR
- added J1: USB4110-GF-A, wsg_fp:USB4110-GF-A_GCT, symbol wsg_syms:USB4110-GF-A
- added L2: 3.3nH, Inductor_SMD:L_0402_1005Metric, symbol Device:L
- added L3: 2.7nH, Inductor_SMD:L_0402_1005Metric, symbol Device:L
- added L4: 2.2nH, Inductor_SMD:L_0402_1005Metric, symbol Device:L
- added R1: 100k, Resistor_SMD:R_0402_1005Metric, symbol Device:R
- added R10, R11: 10k, Resistor_SMD:R_0402_1005Metric, symbol Device:R
- added R2, R3, R4, R5, R6, R7: 0, Resistor_SMD:R_0402_1005Metric, symbol Device:R
- added R8, R9: 5.1k, Resistor_SMD:R_0402_1005Metric, symbol Device:R
- added U2: ESP-PSRAM64H, Package_SO:SOIC-8_3.9x4.9mm_P1.27mm, symbol wsg_syms:1528-4677-ND
- added U3: USBLC6-2SC6, wsg_fp:SOT95P280X145-6N, symbol wsg_syms:USBLC6-2SC6
- added Y2: ECS-.327-12.5-34B-TR, wsg_fp:XTAL_ECS-.327-12.5-34B-TR, symbol wsg_syms:ECS-.327-12.5-34B-TR
- C1, C2: footprint (none) -> Capacitor_SMD:C_0402_1005Metric
- C3, C4: value TBD -> 1.5pF; footprint (none) -> Capacitor_SMD:C_0201_0603Metric
- L1: value TBD -> 2.7nH; footprint (none) -> Inductor_SMD:L_0201_0603Metric
- Y1: footprint ECS-400-10-37B2-CKY-TR:XTAL_ECS-400-10-37B2-CKY-TR -> wsg_fp:XTAL_ECS-400-10-37B2-CKY-TR
Connections:
- net GND is gone; now on net GNDD: C1.1, C2.2, Y1.2, Y1.4
- net GNDA: now reaches C4.1
- net GNDA: now also C3.1, AE1.2 (PCB_Trace), L3.1
- net at L1.2: now also C3.2, C5.2; no longer C4.2
- net at L1.1: now also C4.2, U1.1 (LNA_IN); no longer C3.2
- net CS_FLASH: now reaches U1.15 (GPIO10)
- net CS_FLASH: now also IC2.1 (~{CS}), R1.2
- net MISO_FLASH: now reaches U1.16 (GPIO11)
- net MISO_FLASH: now also IC2.2 (DO_(IO1_))
- net SLCK_FLASH: now reaches U1.17 (GPIO12)
- net SLCK_FLASH: now also IC2.6 (CLK)
- net MOSI_FLASH: now reaches U1.18 (GPIO13)
- net MOSI_FLASH: now also IC2.5 (DI_(IO0_))
- net at U1.2 (VDD3P3), U1.3 (VDD3P3): now also C15.2, L4.2
- net 3V3: now reaches U1.20 (VDD3P3_RTC)
- net 3V3: now also U1.4 (CHIP_PU), U1.46 (VDD3P3_CPU), U1.55 (VDDA), U1.56 (VDDA), C10.2, C11.2, C6.2, C7.2, C8.2, C9.2, IC2.3 (~{WP_(IO2_)}), IC2.7 (~{HOLD_(IO3_)}), IC2.8 (VCC), L4.1, R1.1
- net at U1.21 (XTAL_32K_P): now also C12.2, Y2.2
- net at U1.22 (XTAL_32K_N): now also C13.1, Y2.1
- net at U1.25 (GPIO19/USB_D-): now also U3.3
- net at U1.26 (GPIO20/USB_D+): now also U3.1
- net at U1.28 (SPICS1): now also R2.1
- net VDD_PSRAM: now reaches U1.29 (VDD_SPI)
- net VDD_PSRAM: now also C14.1, U2.8 (Vcc)
- net at U1.30 (SPIHD): now also R3.1
- net at U1.31 (SPIWP): now also R4.1
- net at U1.33 (SPICLK): now also R5.1
- net at U1.34 (SPIQ): now also R6.1
- net at U1.35 (SPID): now also R7.1
- net at U1.5 (GPIO0): now also R11.2
- net at U1.51 (GPIO45): now also U1.52 (GPIO46), R10.1
- net GNDD: now reaches U1.57 (GND)
- net GNDD: now also C10.1, C11.1, C12.1, C13.2, C14.2, C15.1, C6.1, C7.1, C8.1, C9.1, IC2.4 (GND), IC2.9 (EP), J1.A1-B12 (GND), J1.A12-B1 (GND), R10.2, R11.1, R8.2, R9.2, U2.4 (Vss), U3.2
- new net: J1.A5 (CC1), R8.1
- new net: C5.1, L2.1, L3.2
- new net: AE1.1 (FEED), L2.2
- new net: J1.B5 (CC2), R9.1
- new net 5v_USB_EXT: J1.A4-B9 (VBUS), J1.A9-B4 (VBUS), U3.5
- new net CS_PSRAM: R2.2, U2.1 (CE#)
- new net DI_PSRAM: R7.2, U2.5 (SIO[0])
- new net DO_PSRAM: R6.2, U2.2 (SIO[1])
- new net HLD_PSRAM: R3.2, U2.7 (SIO[3])
- new net SCLK_PSRAM: R5.2, U2.6 (SCLK)
- new net USB_D+_EXT: J1.A6 (DP1), J1.B6 (DP2), U3.6
- new net USB_D-_EXT: J1.A7 (DN1), J1.B7 (DN2), U3.4
- new net WP_PSRAM: R4.2, U2.3 (SIO[2])
- no-connect marks 0 -> 3
Other:
- note added: "-->"
- note added: "500R07S1R2BV4T"
- note added: "<--"
- note added: "Bootstrap pins: - GPIO0, GPIO46 - Pulled to GND to allow join bootload mode - GPIO45 - Pulled to GND to make VDD_SPI = 3.3v - GPIO3 - Ignored"
- note added: "CC0402FRNPO9BN120"
- note added: "ESP-PSRAM64H"
- note added: "ESP32-S3FN8"
- note added: "External flash memory will live on SPI2 All other SPI devices will live on SPI3 (SPI3 can be chosen to exist on any of the pins via multiplexing)"
- note added: "GJM1555C1H170FB01D"
- note added: "GRM0335C1H1R5BA01D"
- note added: "Helpful YouTube videos - https://www.youtube.com/watch?v=yxU_Kw2de08 - https://www.youtube.com/watch?v=EdEwRXiQsfc Relevant datasheets: - https://www.espressif.com/sites/default/files/documentation/esp32-s3_datasheet_en.pdf - https://docs.espressif.com/projects/esp-hardware-design-guidelines/en/latest/esp32s3/esp-hardware-design-guidelines-en-master-esp32s3.pdf#page=22&zoom=100,96,580 - https://f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"
- note added: "L-07C2N7SV6T"
- note added: "L-07C3N3SV6T"
- note added: "LQP03TN2N7B02D"
- note added: "NOTES: - SPI3 bus not added yet (can be any four pins) - Expecting a 3V3 rail - 5v coming in from USB (power mux?) - Consider exposing UART* and JTAG pins - Consider adding hardware reset (button to pull pin 4 to GND) - Consider exposing bootstrap pins (buttons or test pads) - Consider adding LEDs (power on+GPIO toggle) *It is recommended to connect a 499 Ω series resistor to the U0TXD line to su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"
- note added: "add a stub to the first capacitor in the matching circuit at the chip end."
- note added: "config me to 3v3 output in fw"
- note added: "hold and wp held high to disable them"
- note added: "this guy is optional if it doesnt fit then delete it i recommend try it first rev to see if extra psram helps at all"
- moved on the sheet: L1, U1
