File: 02-wsg/esp32s3/esp32s3.kicad_pcb (KiCad board)
At the start: 2 copper layers, 36 parts, among them IC2 W25N04KVZEIR, J1 USB4110-GF-A, U1 ESP32-S3, U2 ESP-PSRAM64H, U3 USBLC6-2SC6, Y1 ECS-400-10-37B2-CKY-TR, Y2 ECS-.327-12.5-34B-TR

Commit message: layout first draft
Parts:
- added R10: 10k, Resistor_SMD:R_0402_1005Metric, F.Cu at (106.0, 66.5)
- added R11: 10k, Resistor_SMD:R_0402_1005Metric, F.Cu at (103.3, 66.5)
- moved IC2 58.5 mm to (84.3, 82.4)
- moved Y1 50.1 mm to (100.9, 84.0)
- moved Y2 45.4 mm to (110.0, 81.5), turned to 180 degrees
- moved C1 36.5 mm to (128.0, 67.5)
- moved C8 35.9 mm to (132.3, 67.5)
- moved C12 35.4 mm to (135.8, 67.8)
- moved C2 34.9 mm to (127.3, 71.8)
- moved C9 34.0 mm to (131.5, 72.0)
- moved C13 33.1 mm to (136.3, 72.0)
- moved C6 33.0 mm to (127.5, 75.8)
- moved U3 32.9 mm to (127.8, 96.0)
- moved C10 32.2 mm to (131.5, 76.0)
- moved AE1 32.2 mm to (124.3, 87.0)
- moved C7 31.6 mm to (127.5, 79.5)
- moved J1 31.5 mm to (106.0, 96.0)
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Connections:
- U1 pad 5: unconnected-(U1-GPIO0-Pad5) -> Net-(U1-GPIO0)
- U1 pad 51: unconnected-(U1-GPIO45-Pad51) -> Net-(U1-GPIO45)
- U1 pad 52: unconnected-(U1-GPIO46-Pad52) -> Net-(U1-GPIO45)
