File: 01-main_board/main_board_peripheral_v1/main_board_peripheral_v1.kicad_sch (KiCad schematic)
At the start: 4 parts, among them J1 T4040014041-000, J2 T4040014041-000, J3 0907790004

Commit message: Finished Layout
Parts:
- J3: value 0907790004 -> Mezzanine; footprint 22XT_Main_Peripheral:CONN_SDA-90779_10_MOL -> 22XT_Main_Peripheral:Double Sided Mezzanine Card Edge_Connector Side
Connections:
- net GNDA: now also J3.4 (Pin_4); no longer J3.7 (Pin_7)
- net RX_N: now also J3.10 (Pin_10); no longer J3.3 (Pin_3)
- net RX_P: now also J3.9 (Pin_9); no longer J3.4 (Pin_4)
- net TX_N: now also J3.7 (Pin_7); no longer J3.1 (Pin_1)
- net TX_P: now also J3.6 (Pin_6); no longer J3.2 (Pin_2)
- net USB_D_N: now also J3.2 (Pin_2); no longer J3.9 (Pin_9)
- net USB_D_P: now also J3.1 (Pin_1); no longer J3.8 (Pin_8)
- net USB_5V: now reaches J3.5 (Pin_5)
- net USB_5V: now also F1.2
- removed net 5V_USB: F1.2, J3.10 (Pin_10)
Other:
- note added: "009159010651906"
Changed lines of the file:
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@@
 	(generator_version "9.0")
 	(paper "A4")
+	(text "009159010651906"
+		(exclude_from_sim no)
+		(at 107.696 111.76 0)
+		(effects
+			(font
+				(size 1.27 1.27)
+			)
+		)
+	)
 	(junction
 		(at 85.09 71.12)
@@
 	)
 	(no_connect
-		(at 100.33 97.79)
+		(at 100.33 102.87)
 	)
 	(no_connect
-		(at 100.33 95.25)
+		(at 100.33 90.17)
 	)
 	(wire
@@
 		)
 	)
-	(global_label "RX_P"
+	(global_label "USB_D_P"
 		(shape output)
-		(at 100.33 92.71 180)
-		(fields_autoplaced yes)
-		(effects
-			(font
-				(size 1.27 1.27)
-			)
-			(justify right)
-		)
-		(property "Intersheetrefs" "${INTERSHEET_REFS}"
-			(at 92.6277 92.71 0)
-			(effects
-				(font
-					(size 1.27 1.27)
-				)
-				(justify right)
-				(hide yes)
-			)
-		)
-	)
-	(global_label "USB_D_N"
-		(shape output)
-		(at 100.33 105.41 180)
-		(fields_autoplaced yes)
-		(effects
-			(font
-				(size 1.27 1.27)
-			)
-			(justify right)
-		)
-		(property "Intersheetrefs" "${INTERSHEET_REFS}"
-			(at 88.9991 105.41 0)
+		(at 100.33 85.09 180)
+		(fields_autoplaced yes)
+		(effects
+			(font
+				(size 1.27 1.27)
+			)
+			(justify right)
+		)
+		(property "Intersheetrefs" "${INTERSHEET_REFS}"
+			(at 89.0596 85.09 0)
 			(effects
 				(font
@@
 		)
 	)
-	(global_label "USB_D_P"
-		(shape output)
-		(at 100.33 102.87 180)
-		(fields_autoplaced yes)
-		(effects
-			(font
-				(size 1.27 1.27)
-			)
-			(justify right)
-		)
-		(property "Intersheetrefs" "${INTERSHEET_REFS}"
-			(at 89.0596 102.87 0)
-			(effects
-				(font
-					(size 1.27 1.27)
-				)
-				(justify right)
-				(hide yes)
-			)
-		)
-	)
-	(global_label "5V_USB"
+	(global_label "USB_5V"
 		(shape input)
 		(at 78.74 66.04 180)
@@
 		)
 	)
-	(global_label "RX_N"
-		(shape output)
-		(at 100.33 90.17 180)
-		(fields_autoplaced yes)
-		(effects
-			(font
-				(size 1.27 1.27)
-			)
-			(justify right)
-		)
-		(property "Intersheetrefs" "${INTERSHEET_REFS}"
-			(at 92.5672 90.17 0)
-			(effects
-				(font
-					(size 1.27 1.27)
-				)
-				(justify right)
-				(hide yes)
-			)
-		)
-	)
-	(global_label "TX_P"
-		(shape output)
-		(at 100.33 87.63 180)
-		(fields_autoplaced yes)
-		(effects
-			(font
-				(size 1.27 1.27)
-			)
-			(justify right)
-		)
-		(property "Intersheetrefs" "${INTERSHEET_REFS}"
-			(at 92.9301 87.63 0)
+	(global_label "TX_N"
+		(shape bidirectional)
+		(at 100.33 100.33 180)
+		(fields_autoplaced yes)
+		(effects
+			(font
+				(size 1.27 1.27)
+			)
+			(justify right)
+		)
+		(property "Intersheetrefs" "${INTERSHEET_REFS}"
+			(at 91.7583 100.33 0)
 			(effects
 				(font
@@
 		)
 	)
-	(global_label "TX_N"
+	(global_label "USB_5V"
 		(shape output)
-		(at 100.33 85.09 180)
-		(fields_autoplaced yes)
-		(effects
-			(font
-				(size 1.27 1.27)
-			)
-			(justify right)
-		)
-		(property "Intersheetrefs" "${INTERSHEET_REFS}"
-			(at 92.8696 85.09 0)
-			(effects
-				(font
-					(size 1.27 1.27)
-				)
-				(justify right)
-				(hide yes)
-			)
-		)
-	)
-	(global_label "5V_USB"
-		(shape output)
-		(at 100.33 107.95 180)
-		(fields_autoplaced yes)
-		(effects
-			(font
-				(size 1.27 1.27)
-			)
-			(justify right)
-		)
-		(property "Intersheetrefs" "${INTERSHEET_REFS}"
-			(at 90.2691 107.95 0)
+		(at 100.33 95.25 180)
+		(fields_autoplaced yes)
+		(effects
+			(font
+				(size 1.27 1.27)
+			)
+			(justify right)
+		)
+		(property "Intersheetrefs" "${INTERSHEET_REFS}"
+			(at 90.2691 95.25 0)
+			(effects
+				(font
+					(size 1.27 1.27)
+				)
+				(justify right)
+				(hide yes)
+			)
+		)
+	)
+	(global_label "TX_P"
+		(shape bidirectional)
+		(at 100.33 97.79 180)
+		(fields_autoplaced yes)
+		(effects
+			(font
+				(size 1.27 1.27)
+			)
+			(justify right)
+		)
+		(property "Intersheetrefs" "${INTERSHEET_REFS}"
+			(at 91.8188 97.79 0)
 			(effects
 				(font
@@
 		)
 	)
+	(global_label "USB_D_N"
+		(shape output)
+		(at 100.33 87.63 180)
+		(fields_autoplaced yes)
+		(effects
+			(font
+				(size 1.27 1.27)
+			)
+			(justify right)
+		)
+		(property "Intersheetrefs" "${INTERSHEET_REFS}"
+			(at 88.9991 87.63 0)
+			(effects
+				(font
+					(size 1.27 1.27)
+				)
+				(justify right)
+				(hide yes)
+			)
+		)
+	)
+	(global_label "RX_P"
+		(shape bidirectional)
+		(at 100.33 105.41 180)
+		(fields_autoplaced yes)
+		(effects
+			(font
+				(size 1.27 1.27)
+			)
+			(justify right)
+		)
+		(property "Intersheetrefs" "${INTERSHEET_REFS}"
+			(at 91.5164 105.41 0)
+			(effects
+				(font
+					(size 1.27 1.27)
+				)
+				(justify right)
+				(hide yes)
+			)
+		)
+	)
 	(global_label "TX_N"
 		(shape bidirectional)
@@
 				)
 				(justify left)
+				(hide yes)
+			)
+		)
+	)
+	(global_label "RX_N"
+		(shape bidirectional)
+		(at 100.33 107.95 180)
+		(fields_autoplaced yes)
+		(effects
+			(font
+				(size 1.27 1.27)
+			)
+			(justify right)
+		)
+		(property "Intersheetrefs" "${INTERSHEET_REFS}"
+			(at 91.4559 107.95 0)
+			(effects
+				(font
+					(size 1.27 1.27)
+				)
+				(justify right)
 				(hide yes)
 			)
@@
 	(symbol
 		(lib_id "power:GNDA")
+		(at 100.33 92.71 270)
+		(unit 1)
+		(exclude_from_sim no)
+		(in_bom yes)
+		(on_board yes)
+		(dnp no)
+		(fields_autoplaced yes)
+		(property "Reference" "#PWR01"
+			(at 93.98 92.71 0)
+			(effects
+				(font
+					(size 1.27 1.27)
+				)
+				(hide yes)
+			)
+		)
+		(property "Value" "GNDA"
+			(at 96.52 92.7099 90)
+			(effects
+				(font
+					(size 1.27 1.27)
+				)
+				(justify right)
+			)
+		)
+		(property "Footprint" ""
+			(at 100.33 92.71 0)
+			(effects
+				(font
+					(size 1.27 1.27)
+				)
+				(hide yes)
+			)
+		)
+		(property "Datasheet" ""
+			(at 100.33 92.71 0)
+			(effects
+				(font
+					(size 1.27 1.27)
+				)
+				(hide yes)
+			)
+		)
+		(property "Description" "Power symbol creates a global label with name \"GNDA\" , analog ground"
+			(at 100.33 92.71 0)
+			(effects
+				(font
+					(size 1.27 1.27)
+				)
+				(hide yes)
+			)
+		)
+		(pin "1"
+		)
+		(instances
+			(project ""
+				(path "/e614b84e-efa2-40f7-bc3a-41ecf14c794c"
+					(reference "#PWR01")
+					(unit 1)
+				)
+			)
+		)
+	)
+	(symbol
+		(lib_id "power:GNDA")
 		(at 85.09 71.12 0)
 		(unit 1)
@@
 				(path "/e614b84e-efa2-40f7-bc3a-41ecf14c794c"
 					(reference "#PWR02")
-					(unit 1)
-				)
-			)
-		)
-	)
-	(symbol
-		(lib_id "power:GNDA")
-		(at 100.33 100.33 270)
-		(unit 1)
-		(exclude_from_sim no)
-		(in_bom yes)
-		(on_board yes)
-		(dnp no)
-		(fields_autoplaced yes)
-		(property "Reference" "#PWR01"
-			(at 93.98 100.33 0)
-			(effects
-				(font
-					(size 1.27 1.27)
-				)
-				(hide yes)
-			)
-		)
-		(property "Value" "GNDA"
-			(at 96.52 100.3299 90)
-			(effects
-				(font
-					(size 1.27 1.27)
-				)
-				(justify right)
-			)
-		)
-		(property "Footprint" ""
-			(at 100.33 100.33 0)
-			(effects
-				(font
-					(size 1.27 1.27)
-				)
-				(hide yes)
-			)
-		)
-		(property "Datasheet" ""
-			(at 100.33 100.33 0)
-			(effects
-				(font
-					(size 1.27 1.27)
-				)
-				(hide yes)
-			)
-		)
-		(property "Description" "Power symbol creates a global label with name \"GNDA\" , analog ground"
-			(at 100.33 100.33 0)
-			(effects
-				(font
-					(size 1.27 1.27)
-				)
-				(hide yes)
-			)
-		)
-		(pin "1"
-		)
-		(instances
-			(project ""
-				(path "/e614b84e-efa2-40f7-bc3a-41ecf14c794c"
-					(reference "#PWR01")
 					(unit 1)
 				)
@@
 			)
 		)
-		(property "Value" "0907790004"
+		(property "Value" "Mezzanine"
 			(at 107.95 97.7899 0)
 			(effects
@@
 			)
 		)
-		(property "Footprint" "22XT_Main_Peripheral:CONN_SDA-90779_10_MOL"
+		(property "Footprint" "22XT_Main_Peripheral:Double Sided Mezzanine Card Edge_Connector Side"
 			(at 105.41 95.25 0)
 			(effects
