File: 01-main_board/main_board_v1/main_board_v1.kicad_sch (KiCad schematic)
At the start: 4 parts, among them J1 Mezzanine Edge, J4 DB44 (Analog | Digital)

Commit message: Updating mezz edge
Connections:
- net 5V_usb: now also J1.5 (Pin_5); no longer J1.10 (Pin_10)
- net GNDA: now also J1.4 (Pin_4); no longer J1.9 (Pin_9)
- net RX+: now also J1.9 (Pin_9); no longer J1.4 (Pin_4)
- net RX-: now also J1.10 (Pin_10); no longer J1.5 (Pin_5)
- net TX+: now also J1.6 (Pin_6); no longer J1.1 (Pin_1)
- net TX-: now also J1.7 (Pin_7); no longer J1.2 (Pin_2)
- net usb+: now also J1.1 (Pin_1); no longer J1.6 (Pin_6)
- net usb-: now also J1.2 (Pin_2); no longer J1.7 (Pin_7)
Other:
- note removed: "Picoflex 2x5 Connector"
Changed lines of the file:
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@@
-		)
-	)
-	(text "Picoflex 2x5 Connector\n"
-		(exclude_from_sim no)
-		(at 111.506 29.718 0)
-		(effects
-			(font
-				(size 1.27 1.27)
-			)
 		)
 	)
@@
 		)
 	)
-	(global_label "TX-"
+	(global_label "RX-"
 		(shape bidirectional)
-		(at 111.76 35.56 180)
-		(fields_autoplaced yes)
-		(effects
-			(font
-				(size 1.27 1.27)
-			)
-			(justify right)
-		)
-		(property "Intersheetrefs" "${INTERSHEET_REFS}"
-			(at 103.914 35.56 0)
+		(at 111.76 55.88 180)
+		(fields_autoplaced yes)
+		(effects
+			(font
+				(size 1.27 1.27)
+			)
+			(justify right)
+		)
+		(property "Intersheetrefs" "${INTERSHEET_REFS}"
+			(at 103.6116 55.88 0)
 			(effects
 				(font
@@
 		)
 	)
-	(global_label "usb-"
-		(shape output)
-		(at 111.76 48.26 180)
-		(fields_autoplaced yes)
-		(effects
-			(font
-				(face "KiCad Font")
-				(size 1.27 1.27)
-			)
-			(justify right)
-		)
-		(property "Intersheetrefs" "${INTERSHEET_REFS}"
-			(at 103.8763 48.26 0)
+	(global_label "RX+"
+		(shape bidirectional)
+		(at 111.76 53.34 180)
+		(fields_autoplaced yes)
+		(effects
+			(font
+				(size 1.27 1.27)
+			)
+			(justify right)
+		)
+		(property "Intersheetrefs" "${INTERSHEET_REFS}"
+			(at 103.6116 53.34 0)
 			(effects
 				(font
@@
 		)
 	)
+	(global_label "5V_usb"
+		(shape output)
+		(at 111.76 43.18 180)
+		(fields_autoplaced yes)
+		(effects
+			(font
+				(size 1.27 1.27)
+			)
+			(justify right)
+		)
+		(property "Intersheetrefs" "${INTERSHEET_REFS}"
+			(at 102.183 43.18 0)
+			(effects
+				(font
+					(size 1.27 1.27)
+				)
+				(justify right)
+				(hide yes)
+			)
+		)
+	)
 	(global_label "AN3"
 		(shape input)
@@
 		)
 	)
+	(global_label "usb+"
+		(shape output)
+		(at 111.76 33.02 180)
+		(fields_autoplaced yes)
+		(effects
+			(font
+				(face "KiCad Font")
+				(size 1.27 1.27)
+			)
+			(justify right)
+		)
+		(property "Intersheetrefs" "${INTERSHEET_REFS}"
+			(at 103.8763 33.02 0)
+			(effects
+				(font
+					(size 1.27 1.27)
+				)
+				(justify right)
+				(hide yes)
+			)
+		)
+	)
 	(global_label "DN5"
 		(shape output)
@@
 		)
 	)
+	(global_label "TX+"
+		(shape bidirectional)
+		(at 111.76 45.72 180)
+		(fields_autoplaced yes)
+		(effects
+			(font
+				(size 1.27 1.27)
+			)
+			(justify right)
+		)
+		(property "Intersheetrefs" "${INTERSHEET_REFS}"
+			(at 103.914 45.72 0)
+			(effects
+				(font
+					(size 1.27 1.27)
+				)
+				(justify right)
+				(hide yes)
+			)
+		)
+	)
 	(global_label "5V_buck_PG"
 		(shape input)
@@
 		)
 	)
-	(global_label "RX+"
+	(global_label "TX-"
 		(shape bidirectional)
-		(at 111.76 40.64 180)
-		(fields_autoplaced yes)
-		(effects
-			(font
-				(size 1.27 1.27)
-			)
-			(justify right)
-		)
-		(property "Intersheetrefs" "${INTERSHEET_REFS}"
-			(at 103.6116 40.64 0)
-			(effects
-				(font
-					(size 1.27 1.27)
-				)
-				(justify right)
-				(hide yes)
-			)
-		)
-	)
-	(global_label "RX-"
-		(shape bidirectional)
-		(at 111.76 43.18 180)
-		(fields_autoplaced yes)
-		(effects
-			(font
-				(size 1.27 1.27)
-			)
-			(justify right)
-		)
-		(property "Intersheetrefs" "${INTERSHEET_REFS}"
-			(at 103.6116 43.18 0)
+		(at 111.76 48.26 180)
+		(fields_autoplaced yes)
+		(effects
+			(font
+				(size 1.27 1.27)
+			)
+			(justify right)
+		)
+		(property "Intersheetrefs" "${INTERSHEET_REFS}"
+			(at 103.914 48.26 0)
 			(effects
 				(font
@@
 		)
 	)
-	(global_label "5V_usb"
-		(shape output)
-		(at 111.76 55.88 180)
-		(fields_autoplaced yes)
-		(effects
-			(font
-				(size 1.27 1.27)
-			)
-			(justify right)
-		)
-		(property "Intersheetrefs" "${INTERSHEET_REFS}"
-			(at 102.183 55.88 0)
-			(effects
-				(font
-					(size 1.27 1.27)
-				)
-				(justify right)
-				(hide yes)
-			)
-		)
-	)
-	(global_label "TX+"
-		(shape bidirectional)
-		(at 111.76 33.02 180)
-		(fields_autoplaced yes)
-		(effects
-			(font
-				(size 1.27 1.27)
-			)
-			(justify right)
-		)
-		(property "Intersheetrefs" "${INTERSHEET_REFS}"
-			(at 103.914 33.02 0)
+	(global_label "usb-"
+		(shape output)
+		(at 111.76 35.56 180)
+		(fields_autoplaced yes)
+		(effects
+			(font
+				(face "KiCad Font")
+				(size 1.27 1.27)
+			)
+			(justify right)
+		)
+		(property "Intersheetrefs" "${INTERSHEET_REFS}"
+			(at 103.8763 35.56 0)
 			(effects
 				(font
@@
 				)
 				(justify left)
-				(hide yes)
-			)
-		)
-	)
-	(global_label "usb+"
-		(shape output)
-		(at 111.76 45.72 180)
-		(fields_autoplaced yes)
-		(effects
-			(font
-				(face "KiCad Font")
-				(size 1.27 1.27)
-			)
-			(justify right)
-		)
-		(property "Intersheetrefs" "${INTERSHEET_REFS}"
-			(at 103.8763 45.72 0)
-			(effects
-				(font
-					(size 1.27 1.27)
-				)
-				(justify right)
 				(hide yes)
 			)
@@
 	(symbol
 		(lib_id "power:GND")
-		(at 111.76 53.34 270)
+		(at 111.76 40.64 270)
 		(unit 1)
 		(exclude_from_sim no)
@@
 		(fields_autoplaced yes)
 		(property "Reference" "#PWR038"
-			(at 105.41 53.34 0)
+			(at 105.41 40.64 0)
 			(effects
 				(font
@@
 		)
 		(property "Value" "GNDA"
-			(at 107.95 53.3401 90)
+			(at 107.95 40.6401 90)
 			(effects
 				(font
@@
 		)
 		(property "Footprint" ""
-			(at 111.76 53.34 0)
+			(at 111.76 40.64 0)
 			(effects
 				(font
@@
 		)
 		(property "Datasheet" ""
-			(at 111.76 53.34 0)
+			(at 111.76 40.64 0)
 			(effects
 				(font
@@
 		)
 		(property "Description" "Power symbol creates a global label with name \"GND\" , ground"
-			(at 111.76 53.34 0)
-			(effects
-				(font
+			(at 111.76 40.64 0)
+			(effects
+				(font

Commit message: addressed important drc errors/warnings and added net tie near remaining gnd plane separation
Parts:
- added NT3: NetTie_3_Tee, NetTie:NetTie-3_SMD_Pad0.5mm, symbol Device:NetTie_3_Tee
Connections:
- net GNDA: now also NT3.1; no longer J1.4 (Pin_4)
- net GNDD: now also J1.4 (Pin_4), NT3.2
- net PGND: now also NT3.3

Commit message: added decoupling caps for esp32s3 and resolved drc errors
Parts:
- NT2, NT3: footprint NetTie:NetTie-3_SMD_Pad0.5mm -> NetTie:NetTie-2_SMD_Pad0.5mm
Connections:
- net GNDA: no longer NT3.1
- net PGND: now also NT3.1; no longer NT2.3, NT3.3
Changed lines of the file:
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@@
-	)
-	(symbol
-		(lib_id "power:GNDA")
-		(at 96.52 82.55 0)
-		(unit 1)
-		(exclude_from_sim no)
-		(in_bom yes)
-		(on_board yes)
-		(dnp no)
-		(fields_autoplaced yes)
-		(property "Reference" "#PWR093"
-			(at 96.52 88.9 0)
-			(effects
-				(font
-					(size 1.27 1.27)
-				)
-				(hide yes)
-			)
-		)
-		(property "Value" "PGND"
-			(at 96.52 87.63 0)
-			(effects
-				(font
-					(size 1.27 1.27)
-				)
-			)
-		)
-		(property "Footprint" ""
-			(at 96.52 82.55 0)
-			(effects
-				(font
-					(size 1.27 1.27)
-				)
-				(hide yes)
-			)
-		)
-		(property "Datasheet" ""
-			(at 96.52 82.55 0)
-			(effects
-				(font
-					(size 1.27 1.27)
-				)
-				(hide yes)
-			)
-		)
-		(property "Description" "Power symbol creates a global label with name \"GNDA\" , analog ground"
-			(at 96.52 82.55 0)
-			(effects
-				(font
-					(size 1.27 1.27)
-				)
-				(hide yes)
-			)
-		)
-		(pin "1"
-		)
-		(instances
-			(project "main_board_v1"
-				(path "/12c2237c-5932-49af-9119-92b28c846ae7"
-					(reference "#PWR093")
-					(unit 1)
-				)
-			)
-		)
 	)
 	(symbol
@@
 			)
 		)
-		(property "Footprint" "NetTie:NetTie-3_SMD_Pad0.5mm"
+		(property "Footprint" "NetTie:NetTie-2_SMD_Pad0.5mm"
 			(at 114.3 91.44 0)
 			(effects
@@
 	(symbol
 		(lib_id "power:GNDA")
-		(at 114.3 93.98 0)
-		(unit 1)
-		(exclude_from_sim no)
-		(in_bom yes)
-		(on_board yes)
-		(dnp no)
-		(fields_autoplaced yes)
+		(at 111.76 91.44 270)
+		(unit 1)
+		(exclude_from_sim no)
+		(in_bom yes)
+		(on_board yes)
+		(dnp no)
 		(property "Reference" "#PWR099"
-			(at 114.3 100.33 0)
+			(at 105.41 91.44 0)
 			(effects
 				(font
@@
 		)
 		(property "Value" "PGND"
-			(at 114.3 99.06 0)
+			(at 103.886 92.71 90)
 			(effects
 				(font
@@
 		)
 		(property "Footprint" ""
-			(at 114.3 93.98 0)
+			(at 111.76 91.44 0)
 			(effects
 				(font
@@
 		)
 		(property "Datasheet" ""
-			(at 114.3 93.98 0)
+			(at 111.76 91.44 0)
 			(effects
 				(font
@@
 		)
 		(property "Description" "Power symbol creates a global label with name \"GNDA\" , analog ground"
-			(at 114.3 93.98 0)
+			(at 111.76 91.44 0)
 			(effects
 				(font
@@
 	(symbol
 		(lib_id "power:GNDA")
-		(at 111.76 91.44 270)
-		(unit 1)
-		(exclude_from_sim no)
-		(in_bom yes)
-		(on_board yes)
-		(dnp no)
-		(property "Reference" "#PWR098"
-			(at 105.41 91.44 0)
-			(effects
-				(font
-					(size 1.27 1.27)
-				)
-				(hide yes)
-			)
-		)
-		(property "Value" "GNDA"
-			(at 106.426 90.932 90)
-			(effects
-				(font
-					(size 1.27 1.27)
-				)
-			)
-		)
-		(property "Footprint" ""
-			(at 111.76 91.44 0)
-			(effects
-				(font
-					(size 1.27 1.27)
-				)
-				(hide yes)
-			)
-		)
-		(property "Datasheet" ""
-			(at 111.76 91.44 0)
-			(effects
-				(font
-					(size 1.27 1.27)
-				)
-				(hide yes)
-			)
-		)
-		(property "Description" "Power symbol creates a global label with name \"GNDA\" , analog ground"
-			(at 111.76 91.44 0)
-			(effects
-				(font
-					(size 1.27 1.27)
-				)
-				(hide yes)
-			)
-		)
-		(pin "1"
-		)
-		(instances
-			(project "main_board_v1"
-				(path "/12c2237c-5932-49af-9119-92b28c846ae7"
-					(reference "#PWR098")
-					(unit 1)
-				)
-			)
-		)
-	)
-	(symbol
-		(lib_id "power:GNDA")
 		(at 93.98 80.01 270)
 		(unit 1)
@@
 			)
 		)
-		(property "Footprint" "NetTie:NetTie-3_SMD_Pad0.5mm"
+		(property "Footprint" "NetTie:NetTie-2_SMD_Pad0.5mm"
 			(at 96.52 80.01 0)
 			(effects
