File: 04-dyno_daq/TC_kent/TC_kent.kicad_pcb (KiCad board)
At the start: 2 copper layers, 32.5 x 17 mm, 11 parts, among them J1 Conn_01x04, J2 Conn_01x02, U1 INA333xxDGK

Commit message: Updated grounding for temp pcbs
Routing:
- net GND: vias 5 -> 15
- added copper zone on F.Cu, net GND
Changed lines of the file:
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@@
 			(sketchdnponfab yes)
 			(crossoutdnponfab yes)
-			(subtractmaskfromsilk no)
+			(subtractmaskfromsilk yes)
 			(outputformat 1)
 			(mirror no)
@@
 	)
 	(via
+		(at 125.5 80)
+		(size 0.45)
+		(drill 0.3)
+		(layers "F.Cu" "B.Cu")
+		(net 2)
+	)
+	(via
+		(at 130 91)
+		(size 0.45)
+		(drill 0.3)
+		(layers "F.Cu" "B.Cu")
+		(net 2)
+	)
+	(via
+		(at 133 80)
+		(size 0.45)
+		(drill 0.3)
+		(layers "F.Cu" "B.Cu")
+		(net 2)
+	)
+	(via
+		(at 129.5 80)
+		(size 0.45)
+		(drill 0.3)
+		(layers "F.Cu" "B.Cu")
+		(net 2)
+	)
+	(via
 		(at 142 89.9)
 		(size 0.6)
@@
 	)
 	(via
+		(at 138.5 80)
+		(size 0.45)
+		(drill 0.3)
+		(layers "F.Cu" "B.Cu")
+		(net 2)
+	)
+	(via
+		(at 126 91)
+		(size 0.45)
+		(drill 0.3)
+		(layers "F.Cu" "B.Cu")
+		(net 2)
+	)
+	(via
 		(at 137.9 82.5)
 		(size 0.6)
@@
 		(net 2)
 	)
+	(via
+		(at 133.5 91)
+		(size 0.45)
+		(drill 0.3)
+		(layers "F.Cu" "B.Cu")
+		(net 2)
+	)
+	(via
+		(at 148 80)
+		(size 0.45)
+		(drill 0.3)
+		(layers "F.Cu" "B.Cu")
+		(net 2)
+	)
+	(via
+		(at 139 91)
+		(size 0.45)
+		(drill 0.3)
+		(layers "F.Cu" "B.Cu")
+		(net 2)
+	)
+	(via
+		(at 148.5 91)
+		(size 0.45)
+		(drill 0.3)
+		(layers "F.Cu" "B.Cu")
+		(net 2)
+	)
 	(segment
 		(start 141.5 83.6)
@@
 		(net 2)
 		(net_name "GND")
-		(layer "B.Cu")
+		(layers "F.Cu" "B.Cu")
 		(hatch edge 0.5)
 		(connect_pads
