File: 04-dyno_daq/TC_kent/TC_kent.kicad_sch (KiCad schematic)
At the start: 9 parts, among them J1 Conn_01x04, J2 Conn_01x02, U1 INA333xxDGK

Commit message: Updated grounding for temp pcbs
Other:
- note added: "G=731x"
Changed lines of the file:
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@@
 	(generator_version "9.0")
 	(paper "A4")
+	(text "G=731x"
+		(exclude_from_sim no)
+		(at 111.252 91.44 0)
+		(effects
+			(font
+				(size 1.27 1.27)
+			)
+		)
+	)
 	(junction
 		(at 107.95 86.36)
