File: 01-main_board/main_board_v2/analog_processing.kicad_sch (KiCad schematic)
At the start: 35 parts, among them IC6 AD7175-8BCPZ-RL7

Commit message: made progress on layout
Other:
- moved on the sheet: TP4, TP5, TP6
Changed lines of the file:
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@@
 	(global_label "MISO1"
 		(shape output)
-		(at 115.57 113.03 180)
+		(at 114.3 109.22 180)
 		(fields_autoplaced yes)
 		(effects
@@
 		)
 		(property "Intersheetrefs" "${INTERSHEET_REFS}"
-			(at 106.7791 113.03 0)
+			(at 105.5091 109.22 0)
 			(effects
 				(font
@@
 	(global_label "SCLK1"
 		(shape input)
-		(at 115.57 118.11 180)
+		(at 115.57 119.38 180)
 		(fields_autoplaced yes)
 		(effects
@@
 		)
 		(property "Intersheetrefs" "${INTERSHEET_REFS}"
-			(at 106.5977 118.11 0)
+			(at 106.5977 119.38 0)
 			(effects
 				(font
@@
 	(global_label "MOSI1"
 		(shape input)
-		(at 115.57 115.57 180)
+		(at 115.57 114.3 180)
 		(fields_autoplaced yes)
 		(effects
@@
 		)
 		(property "Intersheetrefs" "${INTERSHEET_REFS}"
-			(at 106.7791 115.57 0)
+			(at 106.7791 114.3 0)
 			(effects
 				(font
@@
 	(symbol
 		(lib_id "Connector:TestPoint")
-		(at 115.57 118.11 270)
+		(at 115.57 119.38 270)
 		(unit 1)
 		(exclude_from_sim no)
@@
 		(fields_autoplaced yes)
 		(property "Reference" "TP6"
-			(at 120.65 116.8399 90)
+			(at 120.65 118.1099 90)
 			(effects
 				(font
@@
 		)
 		(property "Value" "SCLK1"
-			(at 120.65 119.3799 90)
+			(at 120.65 120.6499 90)
 			(effects
 				(font
@@
 		)
 		(property "Footprint" "TestPoint:TestPoint_Pad_1.0x1.0mm"
-			(at 115.57 123.19 0)
+			(at 115.57 124.46 0)
 			(effects
 				(font
@@
 		)
 		(property "Datasheet" "~"
-			(at 115.57 123.19 0)
+			(at 115.57 124.46 0)
 			(effects
 				(font
@@
 		)
 		(property "Description" "test point"
-			(at 115.57 118.11 0)
+			(at 115.57 119.38 0)
 			(effects
 				(font
@@
 	(symbol
 		(lib_id "Connector:TestPoint")
-		(at 115.57 115.57 270)
+		(at 115.57 114.3 270)
 		(unit 1)
 		(exclude_from_sim no)
@@
 		(fields_autoplaced yes)
 		(property "Reference" "TP5"
-			(at 120.65 114.2999 90)
+			(at 120.65 113.0299 90)
 			(effects
 				(font
@@
 		)
 		(property "Value" "MOSI1"
-			(at 120.65 116.8399 90)
+			(at 120.65 115.5699 90)
 			(effects
 				(font
@@
 		)
 		(property "Footprint" "TestPoint:TestPoint_Pad_1.0x1.0mm"
-			(at 115.57 120.65 0)
+			(at 115.57 119.38 0)
 			(effects
 				(font
@@
 		)
 		(property "Datasheet" "~"
-			(at 115.57 120.65 0)
+			(at 115.57 119.38 0)
 			(effects
 				(font
@@
 		)
 		(property "Description" "test point"
-			(at 115.57 115.57 0)
+			(at 115.57 114.3 0)
 			(effects
 				(font
@@
 	(symbol
 		(lib_id "Connector:TestPoint")
-		(at 115.57 113.03 270)
+		(at 114.3 109.22 270)
 		(unit 1)
 		(exclude_from_sim no)
@@
 		(fields_autoplaced yes)
 		(property "Reference" "TP4"
-			(at 120.65 111.7599 90)
+			(at 119.38 107.9499 90)
 			(effects
 				(font
@@
 		)
 		(property "Value" "MISO1"
-			(at 120.65 114.2999 90)
+			(at 119.38 110.4899 90)
 			(effects
 				(font
@@
 		)
 		(property "Footprint" "TestPoint:TestPoint_Pad_1.0x1.0mm"
-			(at 115.57 118.11 0)
+			(at 114.3 114.3 0)
 			(effects
 				(font
@@
 		)
 		(property "Datasheet" "~"
-			(at 115.57 118.11 0)
+			(at 114.3 114.3 0)
 			(effects
 				(font
@@
 		)
 		(property "Description" "test point"
-			(at 115.57 113.03 0)
+			(at 114.3 109.22 0)
 			(effects
 				(font
