File: 01-main_board/DB44_ Breakout/DB44_breakout.kicad_pcb (KiCad board)
At the start: 2 copper layers, 89 x 66.8 mm, 7 parts, among them J1 DB44_Female, J2 Screw_Terminal_01x10 (5.08 mm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, J3 Screw_Terminal_01x10, J4 Screw_Terminal_01x10, J5 Screw_Terminal_01x10, J6 Screw_Terminal_01x04

Commit message: corrected female DB44 footprint
Parts:
- J1: footprint Connector_Dsub:DSUB-44-HD_Socket_Horizontal_P2.29x1.90mm_EdgePinOffset3.03mm_Housed_MountingHolesOffset4.94mm -> 22XT_Main:female-DB44-TE-2311770-1
Routing:
- net Net-(J3-Pin_10): track 64.0 -> 45.2 mm, vias 7 -> 0
- net GND: track 7.29 -> 0.00 mm, vias 51 -> 0
- net Net-(J4-Pin_2): track 55.4 -> 51.8 mm
- net Net-(J5-Pin_6): track 47.9 -> 44.6 mm
- net Net-(J4-Pin_4): track 52.8 -> 49.5 mm
- net Net-(J4-Pin_3): track 53.1 -> 50.6 mm
- net Net-(J5-Pin_9): track 65.0 -> 62.6 mm
- net Net-(J4-Pin_1): track 55.3 -> 52.9 mm, vias 1 -> 0
- net Net-(J5-Pin_10): track 71.9 -> 69.6 mm
- net Net-(J5-Pin_8): track 58.7 -> 56.6 mm
- net Net-(J5-Pin_2): track 39.5 -> 37.5 mm, vias 1 -> 0
- net Net-(J4-Pin_7): track 47.9 -> 46.0 mm
- net Net-(J4-Pin_9): track 46.6 -> 44.7 mm
- net Net-(J3-Pin_9): track 45.7 -> 43.8 mm
- net Net-(J5-Pin_4): track 48.1 -> 50.0 mm
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Other:
- board size 89 x 66.8 mm -> 89 x 69.8 mm
