File: 01-main_board/main_board_v3/teensy.kicad_sch (KiCad schematic)
At the start: 15 parts, among them IC8 AD8591ARTZ-REEL7, U1 Teensy4.1, U3 MCP2562FD-E/SN

Commit message: arranged layout fully, traces almost done, planes wip
Parts:
- C51, C52: value 40pF -> 39pF
- R14, R2: value DNP -> 47
Connections:
- net !LDAC: now also U1.12 (10_CS_MQSR); no longer U1.8 (6_OUT1D)
- net GNDD: no longer U1.58 (GND), U1.59 (GND)
- net LED_CONTROL: now also U1.24 (32_OUT1B); no longer U1.10 (8_TX2_IN1)
- net usb_mux_s: no longer names the net of U1.6 (4_BCLK2)
- no-connect marks 25 -> 28
Changed lines of the file:
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@@
 	)
 	(no_connect
+		(at 182.88 62.23)
+	)
+	(no_connect
 		(at 182.88 49.53)
 	)
 	(no_connect
+		(at 182.88 119.38)
+	)
+	(no_connect
+		(at 182.88 116.84)
+	)
+	(no_connect
 		(at 182.88 54.61)
 	)
@@
 	)
 	(no_connect
+		(at 182.88 52.07)
+	)
+	(no_connect
 		(at 238.76 80.01)
 	)
@@
 	)
 	(no_connect
-		(at 182.88 97.79)
+		(at 182.88 57.15)
 	)
 	(no_connect
@@
 	)
 	(no_connect
-		(at 182.88 67.31)
-	)
-	(no_connect
 		(at 182.88 87.63)
 	)
@@
 	(wire
 		(pts
-			(xy 180.34 57.15) (xy 182.88 57.15)
-		)
-		(stroke
-			(width 0)
-			(type default)
-		)
-	)
-	(wire
-		(pts
 			(xy 242.57 41.91) (xy 238.76 41.91)
 		)
@@
 		)
 	)
-	(global_label "usb_mux_s"
-		(shape input)
-		(at 182.88 52.07 180)
-		(fields_autoplaced yes)
-		(effects
-			(font
-				(size 1.27 1.27)
-			)
-			(justify right)
-		)
-		(property "Intersheetrefs" "${INTERSHEET_REFS}"
-			(at 169.735 52.07 0)
-			(effects
-				(font
-					(size 1.27 1.27)
-				)
-				(justify right)
-				(hide yes)
-			)
-		)
-	)
 	(global_label "D1_shift"
 		(shape input)
@@
 		)
 	)
-	(global_label "LED_CONTROL"
-		(shape output)
-		(at 182.88 62.23 180)
-		(fields_autoplaced yes)
-		(effects
-			(font
-				(size 1.27 1.27)
-			)
-			(justify right)
-		)
-		(property "Intersheetrefs" "${INTERSHEET_REFS}"
-			(at 166.9529 62.23 0)
-			(effects
-				(font
-					(size 1.27 1.27)
-				)
-				(justify right)
-				(hide yes)
-			)
-		)
-	)
 	(global_label "CS_ESP"
 		(shape input)
@@
 		)
 	)
-	(global_label "!LDAC"
-		(shape output)
-		(at 180.34 57.15 180)
-		(fields_autoplaced yes)
-		(effects
-			(font
-				(size 1.27 1.27)
-			)
-			(justify right)
-		)
-		(property "Intersheetrefs" "${INTERSHEET_REFS}"
-			(at 172.0933 57.15 0)
-			(effects
-				(font
-					(size 1.27 1.27)
-				)
-				(justify right)
-				(hide yes)
-			)
-		)
-	)
 	(global_label "5V"
 		(shape input)
@@
 		)
 	)
+	(global_label "LED_CONTROL"
+		(shape output)
+		(at 182.88 97.79 180)
+		(fields_autoplaced yes)
+		(effects
+			(font
+				(size 1.27 1.27)
+			)
+			(justify right)
+		)
+		(property "Intersheetrefs" "${INTERSHEET_REFS}"
+			(at 166.9529 97.79 0)
+			(effects
+				(font
+					(size 1.27 1.27)
+				)
+				(justify right)
+				(hide yes)
+			)
+		)
+	)
 	(global_label "D4_shift"
 		(shape input)
@@
 		)
 	)
+	(global_label "!LDAC"
+		(shape output)
+		(at 182.88 67.31 180)
+		(fields_autoplaced yes)
+		(effects
+			(font
+				(size 1.27 1.27)
+			)
+			(justify right)
+		)
+		(property "Intersheetrefs" "${INTERSHEET_REFS}"
+			(at 174.6333 67.31 0)
+			(effects
+				(font
+					(size 1.27 1.27)
+				)
+				(justify right)
+				(hide yes)
+			)
+		)
+	)
 	(global_label "CTX"
 		(shape input)
@@
 			)
 		)
-		(property "Value" "DNP"
+		(property "Value" "47"
 			(at 253.238 100.838 90)
 			(effects
@@
 	(symbol
 		(lib_id "power:GNDD")
-		(at 182.88 116.84 270)
-		(unit 1)
-		(exclude_from_sim no)
-		(in_bom yes)
-		(on_board yes)
-		(dnp no)
-		(fields_autoplaced yes)
-		(property "Reference" "#PWR043"
-			(at 176.53 116.84 0)
-			(effects
-				(font
-					(size 1.27 1.27)
-				)
-				(hide yes)
-			)
-		)
-		(property "Value" "GNDD"
-			(at 179.07 116.8399 90)
-			(effects
-				(font
-					(size 1.27 1.27)
-				)
-				(justify right)
-			)
-		)
-		(property "Footprint" ""
-			(at 182.88 116.84 0)
-			(effects
-				(font
-					(size 1.27 1.27)
-				)
-				(hide yes)
-			)
-		)
-		(property "Datasheet" ""
-			(at 182.88 116.84 0)
-			(effects
-				(font
-					(size 1.27 1.27)
-				)
-				(hide yes)
-			)
-		)
-		(property "Description" "Power symbol creates a global label with name \"GNDD\" , digital ground"
-			(at 182.88 116.84 0)
-			(effects
-				(font
-					(size 1.27 1.27)
-				)
-				(hide yes)
-			)
-		)
-		(pin "1"
-		)
-		(instances
-			(project "msm"
-				(path "/12c2237c-5932-49af-9119-92b28c846ae7/f7990d3b-6f19-4c8f-ba4f-28eb9e1a3c51"
-					(reference "#PWR043")
-					(unit 1)
-				)
-			)
-		)
-	)
-	(symbol
-		(lib_id "power:GNDD")
 		(at 116.84 111.76 0)
 		(unit 1)
@@
 			)
 		)
-		(property "Value" "40pF"
+		(property "Value" "39pF"
 			(at 133.35 114.2999 0)
 			(effects
@@
 			)
 		)
-		(property "Value" "DNP"
+		(property "Value" "47"
 			(at 252.984 90.17 90)
 			(effects
@@
 	)
 	(symbol
-		(lib_id "power:GNDD")
-		(at 182.88 119.38 270)
-		(unit 1)
-		(exclude_from_sim no)
-		(in_bom yes)
-		(on_board yes)
-		(dnp no)
-		(fields_autoplaced yes)
-		(property "Reference" "#PWR044"
-			(at 176.53 119.38 0)
-			(effects
-				(font
-					(size 1.27 1.27)
-				)
-				(hide yes)
-			)
-		)
-		(property "Value" "GNDD"
-			(at 179.07 119.3799 90)
-			(effects
-				(font
-					(size 1.27 1.27)
-				)
-				(justify right)
-			)
-		)
-		(property "Footprint" ""
-			(at 182.88 119.38 0)
-			(effects
-				(font
-					(size 1.27 1.27)
-				)
-				(hide yes)
-			)
-		)
-		(property "Datasheet" ""
-			(at 182.88 119.38 0)
-			(effects
-				(font
-					(size 1.27 1.27)
-				)
-				(hide yes)
-			)
-		)
-		(property "Description" "Power symbol creates a global label with name \"GNDD\" , digital ground"
-			(at 182.88 119.38 0)
-			(effects
-				(font
-					(size 1.27 1.27)
-				)
-				(hide yes)
-			)
-		)
-		(pin "1"
-		)
-		(instances
-			(project "msm"
-				(path "/12c2237c-5932-49af-9119-92b28c846ae7/f7990d3b-6f19-4c8f-ba4f-28eb9e1a3c51"
-					(reference "#PWR044")
-					(unit 1)
-				)
-			)
-		)
-	)
-	(symbol
 		(lib_id "power:GND")
 		(at 246.38 41.91 90)
@@
 			)
 		)
-		(property "Value" "40pF"
+		(property "Value" "39pF"
 			(at 136.906 96.266 0)
 			(effects

Commit message: finished layout
Connections:
- net !ERROR: now also U1.33 (41_A17); no longer U1.22 (30_CRX3)
Changed lines of the file:
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@@
-	)
-	(no_connect
-		(at 238.76 77.47)
 	)
 	(no_connect
@@
 	(no_connect
 		(at 182.88 90.17)
+	)
+	(no_connect
+		(at 182.88 92.71)
 	)
 	(no_connect
@@
 		)
 	)
-	(global_label "!ERROR"
-		(shape input)
-		(at 182.88 92.71 180)
-		(fields_autoplaced yes)
-		(effects
-			(font
-				(size 1.27 1.27)
-			)
-			(justify right)
-		)
-		(property "Intersheetrefs" "${INTERSHEET_REFS}"
-			(at 173.0005 92.71 0)
-			(effects
-				(font
-					(size 1.27 1.27)
-				)
-				(justify right)
-				(hide yes)
-			)
-		)
-	)
 	(global_label "CRX"
 		(shape output)
@@
 				(hide yes)
 			)
+		)
+	)
+	(global_label "!ERROR"
+		(shape input)
+		(at 238.76 77.47 0)
+		(fields_autoplaced yes)
+		(effects
+			(font
+				(size 1.27 1.27)
+			)
+			(justify left)
+		)
+		(property "Intersheetrefs" "${INTERSHEET_REFS}"
+			(at 248.6395 77.47 0)
+			(effects
+				(font
+					(size 1.27 1.27)
+				)
+				(justify left)
+				(hide yes)
+			)

Commit message: changed peripheral connector, addressed slack revisions
Connections:
- net PGND is gone; now on net GNDD: BT1.2 (-)
- net RESET_DAC: now reaches U1.22 (30_CRX3)
- no-connect marks 28 -> 27
Changed lines of the file:
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@@
-	)
-	(no_connect
-		(at 182.88 92.71)
 	)
 	(no_connect
@@
 		(property "Intersheetrefs" "${INTERSHEET_REFS}"
 			(at 172.8191 72.39 0)
+			(effects
+				(font
+					(size 1.27 1.27)
+				)
+				(justify right)
+				(hide yes)
+			)
+		)
+	)
+	(global_label "RESET_DAC"
+		(shape input)
+		(at 182.88 92.71 180)
+		(fields_autoplaced yes)
+		(effects
+			(font
+				(size 1.27 1.27)
+			)
+			(justify right)
+		)
+		(property "Intersheetrefs" "${INTERSHEET_REFS}"
+			(at 169.5535 92.71 0)
 			(effects
 				(font
@@
 	(symbol
 		(lib_id "power:GNDD")
+		(at 162.56 134.62 0)
+		(unit 1)
+		(exclude_from_sim no)
+		(in_bom yes)
+		(on_board yes)
+		(dnp no)
+		(fields_autoplaced yes)
+		(property "Reference" "#PWR049"
+			(at 162.56 140.97 0)
+			(effects
+				(font
+					(size 1.27 1.27)
+				)
+				(hide yes)
+			)
+		)
+		(property "Value" "GNDD"
+			(at 162.56 138.43 0)
+			(effects
+				(font
+					(size 1.27 1.27)
+				)
+			)
+		)
+		(property "Footprint" ""
+			(at 162.56 134.62 0)
+			(effects
+				(font
+					(size 1.27 1.27)
+				)
+				(hide yes)
+			)
+		)
+		(property "Datasheet" ""
+			(at 162.56 134.62 0)
+			(effects
+				(font
+					(size 1.27 1.27)
+				)
+				(hide yes)
+			)
+		)
+		(property "Description" "Power symbol creates a global label with name \"GNDD\" , digital ground"
+			(at 162.56 134.62 0)
+			(effects
+				(font
+					(size 1.27 1.27)
+				)
+				(hide yes)
+			)
+		)
+		(pin "1"
+		)
+		(instances
+			(project "main_board_v3"
+				(path "/12c2237c-5932-49af-9119-92b28c846ae7/f7990d3b-6f19-4c8f-ba4f-28eb9e1a3c51"
+					(reference "#PWR049")
+					(unit 1)
+				)
+			)
+		)
+	)
+	(symbol
+		(lib_id "power:GNDD")
 		(at 238.76 74.93 90)
 		(unit 1)
@@
 					(unit 1)
 				)
-			)
-		)
-	)
-	(symbol
-		(lib_id "power:GNDA")
-		(at 162.56 134.62 0)
-		(unit 1)
-		(exclude_from_sim no)
-		(in_bom yes)
-		(on_board yes)
-		(dnp no)
-		(property "Reference" "#PWR076"
-			(at 162.56 140.97 0)
-			(effects
-				(font
-					(size 1.27 1.27)
-				)
-				(hide yes)
-			)
-		)
-		(property "Value" "PGND"
-			(at 160.02 140.208 0)
-			(effects
-				(font
-					(size 1.27 1.27)
-				)
-				(justify left)
-			)
-		)
-		(property "Footprint" ""
-			(at 162.56 134.62 0)
-			(effects
-				(font
-					(size 1.27 1.27)
-				)
-				(hide yes)
-			)
-		)
-		(property "Datasheet" ""
-			(at 162.56 134.62 0)
-			(effects
-				(font
-					(size 1.27 1.27)
-				)
-				(hide yes)
-			)
-		)
-		(property "Description" "Power symbol creates a global label with name \"GNDA\" , analog ground"
-			(at 162.56 134.62 0)
-			(effects
-				(font
-					(size 1.27 1.27)
-				)
-				(hide yes)
-			)
-		)
-		(pin "1"
-		)
-		(instances
-			(project "main_board_v1"
-				(path "/12c2237c-5932-49af-9119-92b28c846ae7/f7990d3b-6f19-4c8f-ba4f-28eb9e1a3c51"
-					(reference "#PWR076")
-					(unit 1)
-				)
