File: 01-main_board/main_db44_fpc/main_db44_fpc.kicad_pcb (KiCad board)
At the start: 2 copper layers, 1 part

Commit message: update db44
Parts:
- removed REF**: DSUB-44-HD_Socket_Vertical_P2.29x1.98mm_MountingHoles, Connector_Dsub:DSUB-44-HD_Socket_Vertical_P2.29x1.98mm_MountingHoles
- added FPC_Analog1: Conn_01x24, Connector_FFC-FPC:TE_2-84953-4_1x24-1MP_P1.0mm_Horizontal, F.Cu at (170.0, 101.8)
- added FPC_Digital1: Conn_01x20, Connector_FFC-FPC:TE_2-84953-0_1x20-1MP_P1.0mm_Horizontal, F.Cu at (139.0, 101.8)
- added J1: DB44_Female, jade_moon_footprints:female-DB44-TE-2311770-1-, F.Cu at (139.5, 80.4)
Other:
- copper layers 2 -> 4

Commit message: update db44
Parts:
- added NT1: NetTie_3_Tee, NetTie:NetTie-3_SMD_Pad0.5mm, F.Cu at (153.0, 74.0)
Connections:
- FPC_Analog1 pad MP: (no net) -> GNDA
- FPC_Digital1 pad 20: unconnected-(FPC_Digital1-Pin_20-Pad20) -> GNDD
- FPC_Digital1 pad MP: (no net) -> GNDD
- J1 pad 0: GNDD -> GNDA
- J1 pad 16: unconnected-(J1-Pad16) -> 3V3 Teensy
Routing:
- net AN7: track 0.00 -> 56.9 mm
- net AN10: track 0.00 -> 56.4 mm
- net AN9: track 0.00 -> 55.6 mm
- net 11V1: track 0.00 -> 50.8 mm, vias 0 -> 2
- net AN6: track 0.00 -> 42.5 mm, vias 0 -> 2
- net D4: track 0.00 -> 34.4 mm, vias 0 -> 3
- net sg_sense_1_FL: track 0.00 -> 31.6 mm, vias 0 -> 3
- net GP/Int1: track 0.00 -> 31.2 mm, vias 0 -> 2
- net sg_kelvin_1_FL: track 0.00 -> 31.1 mm, vias 0 -> 3
- net D1: track 0.00 -> 30.2 mm, vias 0 -> 2
- net D6: track 0.00 -> 29.9 mm, vias 0 -> 2
- net AN8: track 0.00 -> 29.7 mm, vias 0 -> 3
- net sg_sense_2_FR: track 0.00 -> 29.3 mm, vias 0 -> 2
- net sg_kelvin_2_FR: track 0.00 -> 27.0 mm, vias 0 -> 3
- net D2: track 0.00 -> 26.0 mm, vias 0 -> 4
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- added copper zone on In2.Cu, net 5V
- added copper zone on In1.Cu, net B-
- added copper zone on In1.Cu, net GNDA
- added copper zone on In1.Cu, net GNDD
Other:
- board outline added: 62 x 38 mm

Commit message: update db44
Routing:
- net AN3: track 0.00 -> 27.1 mm, vias 0 -> 2
- net AN9: track 55.6 -> 32.9 mm, vias 0 -> 2
- net GNDA: track 0.00 -> 20.8 mm, vias 0 -> 13
- net AN7: track 56.9 -> 37.4 mm, vias 0 -> 3
- net D5: track 25.2 -> 43.8 mm, vias 1 -> 0
- net AN10: track 56.4 -> 42.4 mm
- net GNDD: track 6.31 -> 16.3 mm, vias 4 -> 12
- net 11V1: track 50.8 -> 40.9 mm
- net D4: track 34.4 -> 27.7 mm, vias 3 -> 1
- net B-: track 0.39 -> 6.55 mm, vias 0 -> 3
- net AN4: track 22.7 -> 28.3 mm, vias 1 -> 2
- net D6: track 29.9 -> 34.9 mm, vias 2 -> 0
- net GP/Int2: track 22.8 -> 27.2 mm, vias 0 -> 1
- net D1: track 30.2 -> 25.8 mm, vias 2 -> 1
- net AN2: track 22.5 -> 26.2 mm
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
Commit message: update db44
Connections:
- net sg_kelvin_2_FR renamed sg_sense_2_FR-
- net sg_sense_1_FL renamed sg_sense_1_FL+
- FPC_Analog1 pad 8: sg_kelvin_1_FL -> sg_sense_1_FL-
- FPC_Analog1 pad 9: sg_sense_2_FR -> sg_sense_2_FR+
- J1 pad 15: sg_sense_2_FR -> sg_sense_1_FL-
- J1 pad 29: sg_kelvin_1_FL -> sg_sense_2_FR+
Routing:
- net sg_kelvin_1_FL: track 31.4 -> 0.00 mm, vias 2 -> 0
- net sg_sense_2_FR: track 29.2 -> 0.00 mm
- net sg_sense_2_FR+: track 0.00 -> 27.3 mm, vias 0 -> 2
- net sg_sense_1_FL-: track 0.00 -> 20.9 mm, vias 0 -> 2
- net AN7: track 37.4 -> 26.7 mm, vias 3 -> 6
- net sg_sense_1_FL+: track 32.6 -> 23.9 mm, vias 1 -> 0
- net 11V1: track 40.9 -> 48.0 mm, vias 2 -> 1
- net AN6: track 44.8 -> 38.2 mm
- net AN10: track 42.4 -> 37.7 mm, vias 0 -> 2
- net B-: track 6.55 -> 2.21 mm, vias 3 -> 2
- net AN8: track 27.9 -> 30.7 mm, vias 3 -> 2
- net AN5: track 26.6 -> 29.4 mm, vias 2 -> 1
- net sg_sense_2_FR-: track 26.4 -> 24.3 mm, vias 2 -> 3
- net AN3: track 27.1 -> 25.1 mm, vias 2 -> 1
- net AN9: track 32.9 -> 34.7 mm
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
Commit message: Added comments
Connections:
- J1 pad 0: GNDA -> GNDD
Routing:
- net GNDD: track 16.3 -> 18.5 mm, vias 12 -> 13
- net GNDA: track 21.5 -> 19.4 mm, vias 13 -> 12
Other:
- board text added: "NOT a right angle connector"
Changed lines of the file:
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@@
 			(layers "*.Cu" "*.Mask")
 			(remove_unused_layers no)
-			(net 4 "GNDA")
+			(net 20 "GNDD")
 			(pinfunction "MH")
 			(pintype "passive")
@@
 		(layer "Edge.Cuts")
 	)
+	(gr_text "NOT a right angle connector"
+		(at 184.5 68.5 0)
+		(layer "Cmts.User")
+		(effects
+			(font
+				(size 1 1)
+				(thickness 0.15)
+			)
+			(justify left bottom)
+		)
+	)
+	(dimension
+		(type orthogonal)
+		(layer "Cmts.User")
+		(pts
+			(xy 124.5 109.5) (xy 186.5 109.5)
+		)
+		(height 8)
+		(orientation 0)
+		(format
+			(prefix "")
+			(suffix "")
+			(units 3)
+			(units_format 0)
+			(precision 4)
+			(suppress_zeroes yes)
+		)
+		(style
+			(thickness 0.1)
+			(arrow_length 1.27)
+			(text_position_mode 0)
+			(arrow_direction outward)
+			(extension_height 0.58642)
+			(extension_offset 0.5)
+			(keep_text_aligned yes)
+		)
+		(gr_text "62"
+			(at 155.5 116.35 0)
+			(layer "Cmts.User")
+			(effects
+				(font
+					(size 1 1)
+					(thickness 0.15)
+				)
+			)
+		)
+	)
+	(dimension
+		(type orthogonal)
+		(layer "Cmts.User")
+		(pts
+			(xy 124.5 71.5) (xy 124.5 109.5)
+		)
+		(height -21.5)
+		(orientation 1)
+		(format
+			(prefix "")
+			(suffix "")
+			(units 3)
+			(units_format 0)
+			(precision 4)
+			(suppress_zeroes yes)
+		)
+		(style
+			(thickness 0.1)
+			(arrow_length 1.27)
+			(text_position_mode 0)
+			(arrow_direction outward)
+			(extension_height 0.58642)
+			(extension_offset 0.5)
+			(keep_text_aligned yes)
+		)
+		(gr_text "38"
+			(at 101.85 90.5 90)
+			(layer "Cmts.User")
+			(effects
+				(font
+					(size 1 1)
+					(thickness 0.15)
+				)
+			)
+		)
+	)
 	(segment
 		(start 173 85)
@@
 	)
 	(segment
-		(start 131.45 78.475)
-		(end 132.91297 77.01203)
-		(width 0.2)
-		(layer "F.Cu")
-		(net 4)
-	)
-	(segment
 		(start 178.55 78.475)
 		(end 178.55 77.970321)
@@
 	)
 	(segment
-		(start 132.91297 77.01203)
-		(end 133.025506 77.01203)
-		(width 0.2)
-		(layer "F.Cu")
-		(net 4)
-	)
-	(segment
 		(start 153.136 74)
 		(end 154 74.864)
@@
 	(via
 		(at 184.5 100.5)
-		(size 0.6)
-		(drill 0.3)
-		(layers "F.Cu" "B.Cu")
-		(net 4)
-	)
-	(via
-		(at 133.025506 77.01203)
 		(size 0.6)
 		(drill 0.3)
@@
 	)
 	(segment
+		(start 131.45 78.475)
+		(end 132.91297 77.01203)
+		(width 0.2)
+		(layer "F.Cu")
+		(net 20)
+	)
+	(segment
 		(start 134.5 100)
 		(end 134.5 99)
@@
 	)
 	(segment
+		(start 132.91297 77.01203)
+		(end 133.025506 77.01203)
+		(width 0.2)
+		(layer "F.Cu")
+		(net 20)
+	)
+	(segment
 		(start 144.5 100)
 		(end 144.5 101.5)
@@
 		(size 0.6)
 		(drill 0.3)
+		(layers "F.Cu" "B.Cu")
+		(net 20)
+	)
+	(via
+		(at 133.025506 77.01203)
+		(size 0.6)
+		(drill 0.3)

Commit message: update db44
Parts:
- moved NT1 11.2 mm to (151.0, 85.0)
- moved J1 10.5 mm to (138.5, 90.9)
- moved FPC_Digital1 2.52 mm to (136.5, 102.0)
- moved FPC_Analog1 0.50 mm to (169.5, 101.8)
Routing:
- net D5: track 43.8 -> 15.7 mm, vias 0 -> 2
- net D6: track 34.9 -> 13.8 mm, vias 0 -> 2
- net AN7: track 26.7 -> 42.3 mm, vias 6 -> 0
- net GP/Int1: track 28.0 -> 13.0 mm, vias 2 -> 1
- net GP/Int2: track 27.2 -> 12.5 mm, vias 1 -> 3
- net sg_sense_1_FL+: track 23.9 -> 9.72 mm, vias 0 -> 2
- net AN5: track 29.4 -> 15.9 mm
- net sg_sense_2_FR+: track 27.3 -> 15.8 mm, vias 2 -> 3
- net AN4: track 27.1 -> 16.2 mm
- net sg_sense_2_FR-: track 24.3 -> 13.5 mm, vias 3 -> 1
- net sg_sense_1_FL-: track 20.9 -> 10.5 mm, vias 2 -> 0
- net AN1: track 26.8 -> 16.6 mm
- net AN2: track 25.4 -> 15.7 mm
- net AN3: track 25.1 -> 15.9 mm
- net AN9: track 34.7 -> 25.9 mm, vias 2 -> 1
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Other:
- board size 62 x 38 mm -> 65 x 26.5 mm

Commit message: update db44
Routing:
- net sg2_excite: track 2.67 -> 58.3 mm, vias 2 -> 3
- net sg1_excite: track 2.79 -> 50.6 mm, vias 2 -> 3
- net sg_sense_2_FR-: track 13.5 -> 40.7 mm, vias 1 -> 4
- net sg_sense_2_FR+: track 15.8 -> 41.4 mm, vias 3 -> 5
- net AN8: track 32.8 -> 41.8 mm
- net AN6: track 31.0 -> 34.1 mm
- net AN10: track 29.0 -> 30.7 mm
- net AN7: track 42.3 -> 43.8 mm
- net D1: track 27.9 -> 26.6 mm
- net B-: track 3.18 -> 4.39 mm
- net 5V: track 6.16 -> 7.16 mm
- net GNDD: track 18.4 -> 19.1 mm

Commit message: update db44
Routing:
- net sg_sense_1_FL-: track 10.5 -> 12.7 mm
