File: 01-main_board/main_board_peripheral_v3_1/main_board_peripheral_v3_1.kicad_pcb (KiCad board)
At the start: 4 copper layers, 41 x 25 mm, 17 parts, among them J2 T4040014041000, J3 T4041017041-000, J4 FH41-15S-0.5SH_05_, Q1 SSF2302, U1 LM74610QDGKRQ1, U2 MYRBP500080W21RD

Commit message: exported jlcpcb files
Parts:
- added H1: MountingHole, MountingHole:ToolingHole_1.152mm, F.Cu at (133.5, 98.0)
- added H2: MountingHole, MountingHole:ToolingHole_1.152mm, F.Cu at (100.0, 84.0)
