File: 02-wsg/WSG_3.0/WSG_3.0.kicad_pcb (KiCad board)
At the start: 4 copper layers, 48.5 x 23 mm, 103 parts, among them IC1 W25N04KVZEIR, IC10 ESP32-S3, IC2 INA827AIDGK, IC3 MIC5504-3.3YM5-TR, IC4 INA827AIDGK, IC5 GD25Q64ESIG, IC6 INA827AIDGK, IC8 SPX3819S-L_TR, J1 USB4110-GF-A, J2 U.FL-R-SMT-1_10_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

Commit message: finished
Parts:
- removed C13: 1uF, Capacitor_SMD:C_0402_1005Metric
- removed C14: 0.1uF, Capacitor_SMD:C_0402_1005Metric
- removed D2: NHP120SFT3G, Diode_SMD:D_SOD-123F
- removed MOSFET1: SI1317DL-T1-GE3, 22xt_wsg_footprints:SI1317DL-T1-GE3
- removed SW1: SW_Push, wsg_fp:NANOT100AS_butt
- added C27: 0.1uF, Capacitor_SMD:C_0402_1005Metric, F.Cu at (122.8, 82.5)
- added GPIO21: TestPoint, TestPoint:TestPoint_Pad_1.0x1.0mm, B.Cu at (126.8, 80.7)
- added R29: 400, Resistor_SMD:R_0402_1005Metric, B.Cu at (113.1, 80.3)
- added R30: 100k, Resistor_SMD:R_0402_1005Metric, B.Cu at (112.5, 81.5)
- added R31: 0, Resistor_SMD:R_0402_1005Metric, B.Cu at (120.8, 84.5)
- added TP6: TestPoint, TestPoint:TestPoint_Pad_1.0x1.0mm, B.Cu at (118.6, 90.8)
- added U2: TPS2115APWR, 22xt_wsg_footprints:TPS2115APW, B.Cu at (118.0, 81.5)
- C5: value 1pF -> 1.2pF
- C6: value DNP -> 1pF
- C7: value 10pF -> 0.1uF; moved to B.Cu
- L2: value 3.3nH -> 2.4nH
- R27: value DNP -> 100k; moved to B.Cu
- moved R27 15.7 mm to (122.7, 80.6)
- moved C7 12.5 mm to (119.4, 84.6), turned to 90 degrees
- moved C3 5.34 mm to (111.2, 82.7)
- moved C4 5.34 mm to (106.5, 82.5)
- moved R100 5.34 mm to (106.5, 80.6)
- moved R26 5.34 mm to (111.2, 80.8)
- moved SW3 5.34 mm to (113.6, 81.8)
- moved SW4 5.34 mm to (108.8, 82.0)
- moved R45 0.74 mm to (124.5, 83.5)
- moved C29 0.32 mm to (116.2, 84.5), turned to 90 degrees
- moved C11 0.05 mm to (125.0, 93.8)
Connections:
- C29 pad 1: 5.5V_BOOST -> switch_out
- C7 pad 1: GPIO46 -> GND
- C7 pad 2: GND -> 5v_USB_EXT
- IC10 pad 27: unconnected-(IC10-GPIO21-Pad27) -> GPIO21
- IC10 pad 39: unconnected-(IC10-GPIO34-Pad39) -> CS_NAND_FLASH
- IC10 pad 47: CS_NAND_FLASH -> unconnected-(IC10-MTDI-Pad47)
- IC3 pad 1: 5.5V_BOOST -> switch_out
- IC3 pad 3: 5.5V_BOOST -> switch_out
- IC8 pad 1: VIN -> switch_out
- IC8 pad 2: VIN -> switch_out
- R27 pad 1: GPIO46 -> Net-(U2-OUT)
- R27 pad 2: 3V3 -> Net-(U2-STAT)
Routing:
- net 3V3_Ref: track 27.5 -> 46.7 mm, vias 14 -> 15
- net switch_out: track 0.00 -> 18.2 mm, vias 0 -> 2
- net GPIO21: track 0.00 -> 15.4 mm, vias 0 -> 3
- net VIN: track 13.4 -> 0.00 mm
- net Net-(U2-STAT): track 0.00 -> 8.76 mm, vias 0 -> 2
- net 5v_USB_EXT: track 50.1 -> 57.8 mm
- net 5.5V_BOOST: track 12.4 -> 19.6 mm, vias 5 -> 6
- net Net-(U2-OUT): track 0.00 -> 5.94 mm
- net GPIO0: track 41.7 -> 47.2 mm
- net EN: track 38.2 -> 43.4 mm
- net GND: track 111.3 -> 114.3 mm, vias 130 -> 131
- net Net-(U2-ILIM): track 0.00 -> 1.56 mm
- net Net-(IC8-ADJ): track 2.62 -> 4.10 mm
- net CS_NAND_FLASH: track 21.9 -> 20.6 mm
- net GPIO46: track 2.99 -> 1.72 mm
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Other:
- board text removed: "GPIO46"
