File: 02-wsg/WSG_3.0/untitled.kicad_sch (KiCad schematic)
At the start: 31 parts, among them IC1 W25N04KVZEIR, IC3 MIC5504-3.3YM5-TR, IC8 SPX3819S-L_TR, J1 USB4110-GF-A, J4 Conn_01x02, U1 BQ21040DBVR

Commit message: finished
Parts:
- removed C13: 1uF, Capacitor_SMD:C_0402_1005Metric, symbol Device:C
- removed C14: 0.1uF, Capacitor_SMD:C_0402_1005Metric, symbol Device:C
- removed D2: NHP120SFT3G, Diode_SMD:D_SOD-123F, symbol Device:D
- removed MOSFET1: SI1317DL-T1-GE3, 22xt_wsg_footprints:SI1317DL-T1-GE3, symbol 22xt_ICs:DMP2120U-7
- added C27, C7: 0.1uF, Capacitor_SMD:C_0402_1005Metric, symbol Device:C
- added R27, R30: 100k, Resistor_SMD:R_0402_1005Metric, symbol Device:R
- added R29: 400, Resistor_SMD:R_0402_1005Metric, symbol Device:R
- added R31: 0, Resistor_SMD:R_0402_1005Metric, symbol Device:R
- added TP6: TestPoint, TestPoint:TestPoint_Pad_1.0x1.0mm, symbol Connector:TestPoint
- added U2: TPS2115APWR, 22xt_wsg_footprints:TPS2115APW, symbol 22xt_ICs:TPS2115APWR
Connections:
- net 5.5V_BOOST: now also C27.1, TP6.1, U2.6 (IN2); no longer C29.1, IC3.1 (VIN), IC3.3 (EN)
- net 5v_USB_EXT: now also C7.2, R30.1, U2.3 (D1), U2.8 (IN1)
- net GND: now also C27.2, C7.1, R29.2, R30.2, U2.2 (D0), U2.5 (GND)
- net VIN renamed switch_out
- net switch_out: now also C29.1, IC3.1 (VIN), IC3.3 (EN), R31.2
- new net: R27.1, R31.1, U2.7 (OUT)
- new net: R27.2, U2.1 (STAT)
- new net: R29.1, U2.4 (ILIM)
Other:
- note removed: "V_TH_max = -0.8V"
- note removed: "V_fwd_max = 600 mV at 400 mA"
- note removed: "enable pin logic"
- note removed: "include current source"
- note removed: "|V_DS| < |V_GS -V_TH| for triode |4.4| < |0-5.5+0.8|"
- moved on the sheet: C11, C12, IC1, J4, NT1, PS3, R23, R24, R6
