File: 01-main_board/main_board_v4/esp32s3.kicad_sch (KiCad schematic)
At the start: 8 parts, among them U5 XIAO-ESP32-S3

Commit message: regenerated gerbers
Connections:
- net handshake: now reaches U5.2 (GPIO3/A1/D1)
- no-connect marks 3 -> 2
Changed lines of the file:
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@@
-	)
-	(no_connect
-		(at 129.54 88.9)
 	)
 	(no_connect
@@
 				(hide yes)
 			)
+		)
+	)
+	(global_label "handshake"
+		(shape bidirectional)
+		(at 129.54 88.9 180)
+		(fields_autoplaced yes)
+		(effects
+			(font
+				(size 1.27 1.27)
+			)
+			(justify right)
+		)
+		(property "Intersheetrefs" "${INTERSHEET_REFS}"
+			(at 115.4047 88.9 0)
+			(effects
+				(font
+					(size 1.27 1.27)
+				)
+				(justify right)
+				(hide yes)
+			)
