File: 01-main_board/main_board_v4/main_board_v4.kicad_sch (KiCad schematic)
At the start: 10 parts, among them J2 FFC Analog, J3 FFC Digital, J4 FFC Main to Peripheral

Commit message: Added tooling holes
Parts:
- added H5, H6, H7, H8: MountingHole, MountingHole:ToolingHole_1.152mm, symbol Mechanical:MountingHole
Other:
- note added: "Tooling Holes"
