File: 01-main_board/main_board_v4/analog_processing.kicad_sch (KiCad schematic)
At the start: 35 parts, among them IC6 AD7175-8BCPZ-RL7

Commit message: regenerated gerbers
Parts:
- TP4: value MISO1 -> MISO0
- TP5: value MOSI1 -> MOSI0
- TP6: value SCLK1 -> SCLK0
Connections:
- net MISO1 renamed MISO0
- net MOSI1 renamed MOSI0
- net SCLK1 renamed SCLK0
Changed lines of the file:
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@@
 		)
 	)
-	(global_label "SCLK1"
+	(global_label "SCLK0"
 		(shape input)
 		(at 80.01 123.19 270)
@@
 		)
 	)
-	(global_label "MISO1"
+	(global_label "MISO0"
 		(shape output)
 		(at 114.3 109.22 180)
@@
 		)
 	)
-	(global_label "SCLK1"
+	(global_label "SCLK0"
 		(shape input)
 		(at 115.57 119.38 180)
@@
 		)
 	)
-	(global_label "MISO1"
+	(global_label "MISO0"
 		(shape output)
 		(at 74.93 123.19 270)
@@
 		)
 	)
-	(global_label "MOSI1"
+	(global_label "MOSI0"
 		(shape input)
 		(at 77.47 123.19 270)
@@
 		)
 	)
-	(global_label "MOSI1"
+	(global_label "MOSI0"
 		(shape input)
 		(at 115.57 114.3 180)
@@
 			)
 		)
-		(property "Value" "SCLK1"
+		(property "Value" "SCLK0"
 			(at 120.65 120.6499 90)
 			(effects
@@
 			)
 		)
-		(property "Value" "MOSI1"
+		(property "Value" "MOSI0"
 			(at 120.65 115.5699 90)
 			(effects
@@
 			)
 		)
-		(property "Value" "MISO1"
+		(property "Value" "MISO0"
 			(at 119.38 110.4899 90)
 			(effects

Commit message: added nyquist c
meents
Other:
- note added: "edit: sampling at 1 kHz need cutoff frequency <= 500 Hz 0.1 uF, 3.183K ohm"
Changed lines of the file:
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@@
+		)
+	)
+	(text "edit:\nsampling at 1 kHz\nneed cutoff frequency <= 500 Hz\n\n0.1 uF, 3.183K ohm"
+		(exclude_from_sim no)
+		(at 156.972 170.688 0)
+		(effects
+			(font
+				(size 1.27 1.27)
+			)
 		)
 	)
